File: Hardware/MUXUS.kicad_sch (KiCad schematic)
At the start: 124 parts, among them J1 USB_C_Receptacle_USB2.0, J10 USB_A, J2 USB_B, J3 USB_A, J4 USB_B, J5 USB_A, J6 STDC14, J7 SWD, J8 VCP, J9 USB_B, SW1 USER, SW2 RESET, U1 USBLC6-4SC6, U10 AP2151W, U11 AOZ1212AI, U12 USBLC6-2SC6, U13 USBLC6-2SC6, U14 AP2151W, U2 USB2504A-JT, U3 USBLC6-2SC6, U4 USBLC6-2SC6, U5 AP2151W, U6 TS3USBCA420RSVR, U7 STM32G441KBU6, U8 USBLC6-2SC6, U9 USBLC6-2SC6, Y1 ATS240C

Commit message: 67068-9000
Parts:
- J2, J4, J9: footprint 67068-9000:67068-9000 -> leptunKicadLib:67068-9000
Changed lines of the file:
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@@
     (property "Reference" "J2" (id 0) (at 155.1178 16.0782 0))
     (property "Value" "USB_B" (id 1) (at 155.1178 18.3896 0))
-    (property "Footprint" "67068-9000:67068-9000" (id 2) (at 157.48 29.21 0)
+    (property "Footprint" "leptunKicadLib:67068-9000" (id 2) (at 157.48 29.21 0)
       (effects (font (size 1.27 1.27)) hide)
     )
@@
     (property "Reference" "J4" (id 0) (at 244.0178 16.0782 0))
     (property "Value" "USB_B" (id 1) (at 244.0178 18.3896 0))
-    (property "Footprint" "67068-9000:67068-9000" (id 2) (at 246.38 29.21 0)
+    (property "Footprint" "leptunKicadLib:67068-9000" (id 2) (at 246.38 29.21 0)
       (effects (font (size 1.27 1.27)) hide)
     )
@@
     (property "Reference" "J9" (id 0) (at 332.9178 16.0782 0))
     (property "Value" "USB_B" (id 1) (at 332.9178 18.3896 0))
-    (property "Footprint" "67068-9000:67068-9000" (id 2) (at 335.28 29.21 0)
+    (property "Footprint" "leptunKicadLib:67068-9000" (id 2) (at 335.28 29.21 0)
       (effects (font (size 1.27 1.27)) hide)
     )
@@
     )
     (path "/00000000-0000-0000-0000-0000614e1175"
-      (reference "J2") (unit 1) (value "USB_B") (footprint "67068-9000:67068-9000")
+      (reference "J2") (unit 1) (value "USB_B") (footprint "leptunKicadLib:67068-9000")
     )
     (path "/00000000-0000-0000-0000-0000614f9c4f"
@@
     )
     (path "/00000000-0000-0000-0000-00006190b202"
-      (reference "J4") (unit 1) (value "USB_B") (footprint "67068-9000:67068-9000")
+      (reference "J4") (unit 1) (value "USB_B") (footprint "leptunKicadLib:67068-9000")
     )
     (path "/00000000-0000-0000-0000-0000617a921c"
@@
     )
     (path "/00000000-0000-0000-0000-000061927a3b"
-      (reference "J9") (unit 1) (value "USB_B") (footprint "67068-9000:67068-9000")
+      (reference "J9") (unit 1) (value "USB_B") (footprint "leptunKicadLib:67068-9000")
     )
     (path "/00000000-0000-0000-0000-00006185df52"

Commit message: AOZ1212AI
Parts:
- U11: footprint Package_SO:SO-8_3.9x4.9mm_P1.27mm -> leptunKicadLib:AOZ1212AI; symbol AOZ1212AI:AOZ1212AI -> leptunKicadLib:AOZ1212AI
Changed lines of the file:
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@@
     (pin "6")
   )
-  (symbol (lib_id "AOZ1212AI:AOZ1212AI") (at 314.96 162.56 0) (unit 1)
+  (symbol (lib_id "leptunKicadLib:AOZ1212AI") (at 314.96 162.56 0) (unit 1)
     (in_bom yes) (on_board yes)
     (property "Reference" "U11" (id 0) (at 321.31 173.99 0)
@@
       (effects (font (size 1.27 1.27)) (justify left))
     )
-    (property "Footprint" "Package_SO:SO-8_3.9x4.9mm_P1.27mm" (id 2) (at 289.56 151.13 0)
+    (property "Footprint" "leptunKicadLib:AOZ1212AI" (id 2) (at 316.23 186.69 0)
       (effects (font (size 1.27 1.27)) hide)
     )
@@
     )
     (path "/00000000-0000-0000-0000-000061487c04"
-      (reference "U11") (unit 1) (value "AOZ1212AI") (footprint "Package_SO:SO-8_3.9x4.9mm_P1.27mm")
+      (reference "U11") (unit 1) (value "AOZ1212AI") (footprint "leptunKicadLib:AOZ1212AI")
     )
     (path "/00000000-0000-0000-0000-00006185df2c"

Commit message: AP2151W
Parts:
- U10, U14, U5: symbol AP2151W:AP2151W -> leptunKicadLib:AP2151W
Changed lines of the file:
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@@
     (pin "5")
   )
-  (symbol (lib_id "AP2151W:AP2151W") (at 198.12 68.58 0) (mirror y) (unit 1)
+  (symbol (lib_id "leptunKicadLib:AP2151W") (at 198.12 68.58 0) (mirror y) (unit 1)
     (in_bom yes) (on_board yes)
     (property "Reference" "U5" (id 0) (at 198.12 59.2582 0))
@@
     (pin "5")
   )
-  (symbol (lib_id "AP2151W:AP2151W") (at 287.02 68.58 0) (mirror y) (unit 1)
+  (symbol (lib_id "leptunKicadLib:AP2151W") (at 287.02 68.58 0) (mirror y) (unit 1)
     (in_bom yes) (on_board yes)
     (property "Reference" "U10" (id 0) (at 287.02 59.2582 0))
@@
     (pin "5")
   )
-  (symbol (lib_id "AP2151W:AP2151W") (at 375.92 68.58 0) (mirror y) (unit 1)
+  (symbol (lib_id "leptunKicadLib:AP2151W") (at 375.92 68.58 0) (mirror y) (unit 1)
     (in_bom yes) (on_board yes)
     (property "Reference" "U14" (id 0) (at 375.92 59.2582 0))

Commit message: DTSM-61N-V-T_R
Parts:
- SW1, SW2: footprint Button_Switch_SMD:SW_Push_1P1T_NO_6x6mm_H9.5mm -> leptunKicadLib:DTSM-61N-V-T_R
Changed lines of the file:
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@@
     (property "Reference" "SW1" (id 0) (at 259.08 232.791 0))
     (property "Value" "USER" (id 1) (at 259.08 235.1024 0))
-    (property "Footprint" "Button_Switch_SMD:SW_Push_1P1T_NO_6x6mm_H9.5mm" (id 2) (at 259.08 234.95 0)
+    (property "Footprint" "leptunKicadLib:DTSM-61N-V-T_R" (id 2) (at 259.08 234.95 0)
       (effects (font (size 1.27 1.27)) hide)
     )
@@
     (property "Reference" "SW2" (id 0) (at 259.08 264.541 0))
     (property "Value" "RESET" (id 1) (at 259.08 266.8524 0))
-    (property "Footprint" "Button_Switch_SMD:SW_Push_1P1T_NO_6x6mm_H9.5mm" (id 2) (at 259.08 266.7 0)
+    (property "Footprint" "leptunKicadLib:DTSM-61N-V-T_R" (id 2) (at 259.08 266.7 0)
       (effects (font (size 1.27 1.27)) hide)
     )
@@
     )
     (path "/00000000-0000-0000-0000-000061d2f89d"
-      (reference "SW1") (unit 1) (value "USER") (footprint "Button_Switch_SMD:SW_Push_1P1T_NO_6x6mm_H9.5mm")
+      (reference "SW1") (unit 1) (value "USER") (footprint "leptunKicadLib:DTSM-61N-V-T_R")
     )
     (path "/00000000-0000-0000-0000-000061dd83f5"
-      (reference "SW2") (unit 1) (value "RESET") (footprint "Button_Switch_SMD:SW_Push_1P1T_NO_6x6mm_H9.5mm")
+      (reference "SW2") (unit 1) (value "RESET") (footprint "leptunKicadLib:DTSM-61N-V-T_R")
     )
     (path "/00000000-0000-0000-0000-0000615445ff"

Commit message: rev2 dump
Parts:
- removed C12, C17, C21: 100nF, Capacitor_SMD:C_0805_2012Metric, symbol Device:C_Small
- removed C16: 1uF, Capacitor_SMD:C_0805_2012Metric, symbol Device:C_Small
- removed C19, C23, C24, C32, C34, C35, C36, C38, C40: 100nF, Capacitor_SMD:C_0805_2012Metric, symbol Device:C
- removed C28, C37: 120uF, Capacitor_THT:C_Radial_D6.3mm_H11.0mm_P2.50mm, symbol Device:C
- removed C30, C39: 22uF, Capacitor_SMD:C_1210_3225Metric, symbol Device:C
- removed C31: 1uF, Capacitor_SMD:C_0805_2012Metric, symbol Device:C
- removed C33: 100pF, Capacitor_SMD:C_0805_2012Metric, symbol Device:C
- removed D10, D11, D12: LED, LED_THT:LED_D5.0mm, symbol Device:LED
- removed D13: B540C-13-F, Diode_SMD:D_SMC, symbol Device:D_Schottky
- removed H2, H3, H4: MountingHole_Pad, MountingHole:MountingHole_3.2mm_M3_Pad_Via, symbol Mechanical:MountingHole_Pad
- removed J1: USB_C_Receptacle_USB2.0, leptunKicadLib:USB4110-GF-A, symbol Connector:USB_C_Receptacle_USB2.0
- removed J10, J3, J5: USB_A, leptunKicadLib:67643-0910, symbol Connector:USB_A
- removed J2, J4, J9: USB_B, leptunKicadLib:67068-9000, symbol Connector:USB_B
- removed J7: SWD, Connector_PinHeader_2.54mm:PinHeader_1x06_P2.54mm_Vertical, symbol Connector_Generic:Conn_01x06
- removed J8: VCP, Connector_PinHeader_2.54mm:PinHeader_1x02_P2.54mm_Vertical, symbol Connector_Generic:Conn_01x02
- removed L1: SRP6530A-6R8M, leptunKicadLib:SRP6530A-6R8M, symbol Device:L
- removed R1, R18, R26: 330R, Resistor_SMD:R_0805_2012Metric, symbol Device:R
- removed R2: 10K, Resistor_SMD:R_1206_3216Metric, symbol Device:R
- removed R21, R22, R23, R24: 100R, Resistor_SMD:R_0805_2012Metric, symbol Device:R
- removed R25: 15K, Resistor_SMD:R_1206_3216Metric, symbol Device:R
- removed R28: 31.6K, Resistor_SMD:R_1206_3216Metric, symbol Device:R_Small
- removed R29: 10K, Resistor_SMD:R_1206_3216Metric, symbol Device:R_Small
- removed R3: 1K, Resistor_SMD:R_1206_3216Metric, symbol Device:R
- removed U1: USBLC6-4SC6, Package_TO_SOT_SMD:SOT-23-6, symbol Power_Protection:USBLC6-4SC6
- removed U10, U14, U5: AP2151W, Package_TO_SOT_SMD:SOT-23-5, symbol leptunKicadLib:AP2151W
- removed U11: AOZ1212AI, leptunKicadLib:AOZ1212AI, symbol leptunKicadLib:AOZ1212AI
- removed U12, U13, U4, U8, U9: USBLC6-2SC6, Package_TO_SOT_SMD:SOT-23-6, symbol Power_Protection:USBLC6-2SC6
- removed U6: TS3USBCA420RSVR, leptunKicadLib:TS3USBCA420RSVR, symbol leptunKicadLib:TS3USBCA420RSVR
- removed U7: STM32G441KBU6, leptunKicadLib:STM32G441KBU6, symbol leptunKicadLib:STM32G441KBU6
- added C11, C16, C2, C5, C7, C8: 100nF, Capacitor_SMD:C_0805_2012Metric, symbol Device:C
- added C15, C17: 120uF, Capacitor_THT:C_Radial_D6.3mm_H11.0mm_P2.50mm, symbol Device:C
- added C19: 4.7uF, Capacitor_SMD:C_1206_3216Metric, symbol Device:C_Small
- added C24, C25, C26, C27, C31, C37: 100nF, Capacitor_SMD:C_0805_2012Metric, symbol Device:C_Small
- added C9: 22uF, Capacitor_SMD:C_1210_3225Metric, symbol Device:C
- added D2, D3, D4: BLUE, LED_SMD:LED_1206_3216Metric, symbol Device:LED
- added J1: 33UBAR-TSN1R, leptunKicadLib:33UBAR-TSN1R, symbol leptunKicadLib:33UBAR-TSN1R
- added J2, J3, J4, J5: USB4110-GF-A, leptunKicadLib:USB4110-GF-A, symbol Connector:USB_C_Receptacle_USB2.0
- added JP1: DBCC1, Jumper:SolderJumper-3_P1.3mm_Bridged12_RoundedPad1.0x1.5mm_NumberLabels, symbol Jumper:SolderJumper_3_Bridged12
- added R10, R15, R7, R8, R9: 5.1K, Resistor_SMD:R_0603_1608Metric, symbol Device:R
- added R12, R13, R5, R6: 330R, Resistor_SMD:R_0805_2012Metric, symbol Device:R
- added R16, R28, R29, R30, R32, R33: 10K, Resistor_SMD:R_0805_2012Metric, symbol Device:R
- added R42: 1M, Resistor_SMD:R_0603_1608Metric, symbol Device:R
- added U1, U2, U5: USBLC6-2SC6, Package_TO_SOT_SMD:SOT-23-6, symbol Power_Protection:USBLC6-2SC6
- added U11, U9: PI3USB102, Package_DFN_QFN:UQFN-10_1.4x1.8mm_P0.4mm, symbol leptunKicadLib:PI3USB102
- added U4: LD1117S33CTR, Package_TO_SOT_SMD:SOT-223-3_TabPin2, symbol Regulator_Linear:LD1117S33TR_SOT223
- added U6: TPS2053BDR, leptunKicadLib:TPS2053BDR, symbol leptunKicadLib:TPS2053BDR
- added U7: MC74VHC1G08DBVT1G, leptunKicadLib:MC74VHC1G08DBVT1G, symbol 74xGxx:74AHC1G08
- added U8: STM32G0B1KET6N, Package_QFP:LQFP-32_7x7mm_P0.8mm, symbol leptunKicadLib:STM32G0B1KET6N
- C22: renamed from C2; value 15pF -> 33pF; footprint Capacitor_SMD:C_0805_2012Metric -> Capacitor_SMD:C_0603_1608Metric
- C23: renamed from C1; value 15pF -> 33pF; footprint Capacitor_SMD:C_0805_2012Metric -> Capacitor_SMD:C_0603_1608Metric
- D1: renamed from D9; value LED -> BLUE; footprint LED_THT:LED_D5.0mm -> LED_SMD:LED_1206_3216Metric
- R11: renamed from R20; footprint Resistor_SMD:R_1206_3216Metric -> Resistor_SMD:R_0805_2012Metric
- R14: value 330R -> 5.1K; footprint Resistor_SMD:R_0805_2012Metric -> Resistor_SMD:R_0603_1608Metric
- R17, R27: value 330R -> 10K
- R18: renamed from R30; footprint Resistor_SMD:R_1206_3216Metric -> Resistor_SMD:R_0805_2012Metric
- R19: renamed from R31; footprint Resistor_SMD:R_1206_3216Metric -> Resistor_SMD:R_0805_2012Metric
- R2: renamed from R16; value 1K -> 10K; footprint Resistor_SMD:R_1206_3216Metric -> Resistor_SMD:R_0805_2012Metric
- R20: renamed from R32; footprint Resistor_SMD:R_1206_3216Metric -> Resistor_SMD:R_0805_2012Metric
- R21: renamed from R33; footprint Resistor_SMD:R_1206_3216Metric -> Resistor_SMD:R_0805_2012Metric
- R22: renamed from R34; footprint Resistor_SMD:R_1206_3216Metric -> Resistor_SMD:R_0805_2012Metric
- R23: renamed from R35; footprint Resistor_SMD:R_1206_3216Metric -> Resistor_SMD:R_0805_2012Metric
- R24: renamed from R36; footprint Resistor_SMD:R_1206_3216Metric -> Resistor_SMD:R_0805_2012Metric
- R25: renamed from R37; footprint Resistor_SMD:R_1206_3216Metric -> Resistor_SMD:R_0805_2012Metric
- R3: renamed from R15; value 1K -> 10K; footprint Resistor_SMD:R_1206_3216Metric -> Resistor_SMD:R_0805_2012Metric
- R4: renamed from R19; footprint Resistor_SMD:R_1206_3216Metric -> Resistor_SMD:R_0805_2012Metric
- SW1, SW2: footprint leptunKicadLib:DTSM-61N-V-T_R -> leptunKicadLib:FSM4JSMAATR
- renumbered C13 to C1, C18 to C10, C29 to C12, C15 to C13, C20 to C18, C22 to C20, C25 to C21, C7 to C28, C6 to C29, C8 to C30, C9 to C32, C10 to C33, C11 to C34, C5 to C35, C4 to C36, C26 to C4, C27 to C6, D6 to D10, D7 to D11, D8 to D12, D1 to D5, D2 to D6, D3 to D7, D4 to D8, D5 to D9, R12 to R1, R4 to R26, R5 to R34, R6 to R35, R7 to R36, R8 to R37, R9 to R38, R10 to R39, R11 to R40, R13 to R41, U2 to U10
Connections:
- net +3V3: now also C35.2, C36.2, D1.2 (A), C19.1, C31.1, C37.1, C9.1, D2.2 (A), D3.2 (A), D4.2 (A), R16.2, R29.2, R30.2, R32.2, R33.2, U11.9 (VDD), U4.2 (VO), U7.5 (VCC), U8.20 (VDDIO2), U8.4 (VDD/VDDA), U9.9 (VDD); no longer U10.62 (ATEST/REG_EN)
- net CC1: now also JP1.2 (C), U5.1 (I/O1), U8.26 (PD0)
- net CC2: now also U5.3 (I/O2), U8.28 (PD2), U8.29 (PD3)
- net DFP1_D+: now also U8.23 (PA12_[PA10])
- net DFP1_D-: now also U8.22 (PA11_[PA9])
- net DFP2_CONN_D+: now also J1.3 (D1+), U1.1 (I/O1); no longer U3.3 (I/O2)
- net DFP2_CONN_D-: now also J1.2 (D1-), U1.3 (I/O2); no longer U3.1 (I/O1)
- net DFP2_D+: now also U1.6 (I/O1); no longer U3.4 (I/O2)
- net DFP2_D-: now also U1.4 (I/O2); no longer U3.6 (I/O1)
- net DFP2_EN: now also U6.3 (EN1)
- net DFP2_OCSn: now also U6.16 (nOC1)
- net DFP3_CONN_D+: now also J1.7 (D2+), U2.1 (I/O1)
- net DFP3_CONN_D-: now also J1.6 (D2-), U2.3 (I/O2)
- net DFP3_D+: now also U2.6 (I/O1)
- net DFP3_D-: now also U2.4 (I/O2)
- net DFP3_EN: now also U6.4 (EN2)
- net DFP3_OCSn: now also U6.13 (nOC2)
- net DFP4_CONN_D+: now also U3.3 (I/O2), J1.11 (D3+)
- net DFP4_CONN_D-: now also U3.1 (I/O1), J1.10 (D3-)
- net DFP4_D+: now also U3.4 (I/O2)
- net DFP4_D-: now also U3.6 (I/O1)
- net DFP4_EN: now also U6.7 (EN3)
- net DFP4_OCSn: now also U6.12 (nOC3)
- net GND: now also C23.1, C3.2, R14.1, C11.2, C15.2, C16.2, C17.2, C19.2, C2.2, C24.1, C25.1, C26.1, C27.1, C31.2, C37.2, C5.2, C7.2, C8.2, C9.2, J1.12 (GND3), J1.4 (GND1), J1.8 (GND2), J2.A1 (GND), J2.A12 (GND), J2.B1 (GND), J2.B12 (GND), J3.A1 (GND), J3.A12 (GND), J3.B1 (GND), J3.B12 (GND), J4.A1 (GND), J4.A12 (GND), J4.B1 (GND), J4.B12 (GND), J5.A1 (GND), J5.A12 (GND), J5.B1 (GND), J5.B12 (GND), R10.1, R12.2, R13.2, R15.1, R28.2, R5.2, R6.2, R7.1, R8.1, R9.1, U1.2 (GND), U11.3 (GND), U2.2 (GND), U4.1 (GND), U5.2 (GND), U6.1 (GND), U6.5 (GND), U7.3 (GND), U8.5 (VSS/VSSA), U9.3 (GND); no longer C23.2, C3.1, R14.2, R17.1
- net HUB_RESET: now also R30.1, U8.1 (PB9)
- net I2C1_SCL: now also R2.2, U8.30 (PB6); no longer R3.2
- net I2C1_SDA: now also R3.2, U8.31 (PB7); no longer R2.2
- net IFP_D+: now also U11.2 (Y-), U9.2 (Y-)
- net IFP_D-: now also U11.1 (Y+), U9.1 (Y+)
- net IFP_VBUS: now also R29.1, U8.32 (PB8)
- net LED1: now also U8.16 (PB1)
- net LED2: now also D2.1 (K), U8.15 (PB0)
- net LED3: now also D3.1 (K), U8.17 (PB15)
- net LED4: now also D4.1 (K), U8.19 (PA9)
- net LPUART1_RX: now also U8.10 (PA3)
- net LPUART1_TX: now also U8.9 (PA2)
- net NRST: now also U8.6 (PF2-NRST)
- net SWCLK: now also R17.2, U8.25 (PA14-BOOT0)
- net SWDIO: now also U8.24 (PA13)
- net UFP1_D+: now also J5.A6 (D+), J5.B6 (D+), U9.4 (M-)
- net UFP1_D-: now also J5.A7 (D-), J5.B7 (D-), U9.5 (M+)
- net UFP2_D+: now also J3.A6 (D+), J3.B6 (D+), U9.6 (D-)
- net UFP2_D-: now also J3.A7 (D-), J3.B7 (D-), U9.7 (D+)
- net UFP2_VBUS: now also J3.A4 (VBUS), J3.A9 (VBUS), J3.B4 (VBUS), J3.B9 (VBUS)
- net UFP3_D+: now also J4.A6 (D+), J4.B6 (D+), U11.4 (M-)
- net UFP3_D-: now also J4.A7 (D-), J4.B7 (D-), U11.5 (M+)
- net UFP3_VBUS: now also J4.A4 (VBUS), J4.A9 (VBUS), J4.B4 (VBUS), J4.B9 (VBUS)
- net UFP4_D+: now also J2.A6 (D+), J2.B6 (D+), U11.6 (D-)
- net UFP4_D-: now also J2.A7 (D-), J2.B7 (D-), U11.7 (D+)
- net UFP4_VBUS: now also J2.A4 (VBUS), J2.A9 (VBUS), J2.B4 (VBUS), J2.B9 (VBUS)
- net VBUS: now also C10.1, C11.1, J5.A4 (VBUS), J5.A9 (VBUS), J5.B4 (VBUS), J5.B9 (VBUS), U5.5 (VBUS), U6.2 (IN1), U6.6 (IN2)
- net VOLT1: now also U8.11 (PA4)
- net VOLT2: now also U8.12 (PA5)
- net VOLT3: now also U8.13 (PA6)
- net VOLT4: now also U8.14 (PA7)
- net at F1.1: now also C5.1, U4.3 (VI)
- net DFP3_VBUS: now reaches C14.1
- net DFP3_VBUS: now also C15.1, J1.5 (VBUS2), U2.5 (VBUS), U6.14 (OUT2); no longer R14.1
- net at C1.2, R1.2: now also J1.0 (Shield)
- net at C22.2, U10.58 (XTAL1/CLKIN): now also Y1.1, R42.1; no longer Y1.2
- net at U10.30 (VDD18): now also C29.2, U10.42 (VDD18), U10.54 (VDD18), C24.2, C25.2, C26.2; no longer C36.2
- net at C28.2, U10.60 (VDDA18PLL): now also C27.2
- net DFP2_VBUS: now reaches C12.1
- net DFP2_VBUS: now also C13.1, J1.1 (VBUS1), U1.5 (VBUS), U6.15 (OUT1)
- net MUX_EN1: now reaches R27.1
- net MUX_EN1: now also U8.7 (PA0), U9.8 (nOE)
- net GNDDetect: now reaches J6.11 (Pin_11)
- net GNDDetect: now also R16.1, U7.1
- net BOOT0 renamed USER
- net USER: now also U7.2, U8.18 (PA8)
- net SWO: no longer names the net of J6.8 (Pin_8)
- new net: C23.2, R42.2, U10.57 (XTAL2), Y1.2
- new net: R33.1, U10.62 (ATEST/REG_EN)
- new net: J2.A5 (CC1), R7.2
- new net: J2.B5 (CC2), R8.2
- new net: C2.1, J2.S1 (SHIELD), R5.1
- new net: J3.B5 (CC2), R10.2
- new net: R17.1, U7.4
- new net: C7.1, J4.S1 (SHIELD), R12.1
- new net: J5.A5 (CC1), U5.6 (I/O1)
- new net: J5.B5 (CC2), U5.4 (I/O2)
- new net: C8.1, J5.S1 (SHIELD), R13.1
- new net: J4.B5 (CC2), R15.2
- new net: C3.1, J3.S1 (SHIELD), R6.1
- new net: J3.A5 (CC1), R9.2
- new net: J4.A5 (CC1), R14.2
- new net DFP4_VBUS: C16.1, C17.1, J1.9 (VBUS3), U3.5 (VBUS), U6.11 (OUT3)
- new net MUX_EN2: R32.1, U11.8 (nOE), U8.8 (PA1)
- new net MUX_SEL: R28.1, U11.10 (SEL), U8.2 (PC14-OSC32_IN), U9.10 (SEL)
- new net REPLACEMENT_UCPD2_DBCC1: JP1.1 (A), U8.21 (PA10)
- new net RESERVED_UCPD2_DBCC1: JP1.3 (B), U8.27 (PD1)
- no-connect marks 14 -> 24
Other:
- note added: "3.3V rail LDO"
- note added: "AMOGUS"
- note added: "BOOT0_LOGIC"
- note added: "Buttons"
- note added: "DFP ESD protection"
- note added: "DFP power switch"
- note added: "Downstream USB ports"
- note added: "I2C pullup resistors"
- note added: "MCU"
- note added: "MCU LEDs"
- note added: "MCU Programming header"
- note added: "MISC"
- note added: "MUX"
- note added: "Parts inventory"
- note added: "Passive pin states"
- note added: "UFP VBUS ADC voltage dividers"
- note added: "USB HUB"
- note added: "Upstream USB ports"
- title: (none) -> MUXUS
- moved on the sheet: C1, C10, C12, C13, C18, C20, C21, C22, C23, C28, C29, C30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
